File: Kicad/exp_card/exp_card.sch (KiCad schematic (older format))
At the start: 1 part

Commit message: update
Parts:
- gave numbers to parts that had none: 1
Changed lines of the file:
@@
 $EndDescr
 $Comp
-L !MyLib:maxim_exp_slot U?
+L !MyLib:maxim_exp_slot U1
 U 1 1 6092FEF3
 P 4100 3500
-F 0 "U?" H 4125 5715 50  0000 C CNN
+F 0 "U1" H 4125 5715 50  0000 C CNN
 F 1 "maxim_exp_slot" H 4125 5624 50  0000 C CNN
 F 2 "!mymodules:maxim_exp_card_narrow_flipped" H 2000 4950 50  0001 C CNN
